File: eagle/Segment16Keyboard.brd (EAGLE design)
At the start: 56.1 x 27.5 mm, 6 parts, among them U1 LCD-16X2NOHOLES

Commit message: WIP
Parts:
- added C1, C2, C3: 0.1uF, adafruit:C0805
- added C10: 0.1uF, resistor:C0805
- added C13, C19: 10uF, resistor:C0805
- added D3: Green, adafruit:CHIPLED_0805
- added ISP_V13: (no value), SparkFun-Connectors:1X06
- added JP2: FTDI Basic, SparkFun:1X06
- added LED1: Red, Testing:0603-LED-ALT1
- added Q1: 16MHZ, SparkFun-FreqCtrl:RESONATOR-SMD
- added R11: 10K, SparkFun:0603-RES
- added R2: 10K, adafruit:M0805
- added R6: 300, adafruit:M0805
- added S1: Reset, Testing:TACTILE-SWITCH-SMD-ALT01
- added SJ1: (no value), SparkFun-Passives:SJ_2S
- added U2: ATMEGA328, SparkFun:TQFP32-08
- added U3: MIC5205, SparkFun:SOT23-5
Connections:
- new net A0: U2.23
- new net A1: U2.24
- new net A2: U2.25
- new net A3: U2.26
- new net A4: U2.27
- new net A5: U2.28
- new net A6: U2.19
- new net A7: U2.22
- new net AREF: C1.2, U2.20
- new net D10: U2.14
- new net D2: U2.32
- new net D3: U2.1
- new net D4: U2.2
- new net D5: U2.9
- new net D6: U2.10
- new net D7: U2.11
- new net DTR: C2.2, JP2.1
- new net MISO: ISP_V13.3, U2.16
- new net MOSI: ISP_V13.2, U2.15
- new net N$12: D3.A, R6.2
- new net N$13: Q1.3, U2.8
- new net N$15: Q1.1, U2.7
- new net N$19: LED1.A, SJ1.1, U3.5
- new net N$20: LED1.C, R11.2
- new net RESET: C2.1, ISP_V13.1, R2.1, S1.3, S1.4, U2.29
- new net RXI: JP2.3, U2.30
- new net SCK: ISP_V13.5, R6.1, U2.17
- new net SSRX: U2.12
- new net SSTX: U2.13
- new net TXO: JP2.2, U2.31
- new net VCC: C10.1, C13.1, C3.2, ISP_V13.4, JP2.4, R2.2, SJ1.2, U2.18, U2.4, U2.6
- net GND: now also C1.1, C10.2, C13.2, C19.2, C3.1, D3.C, ISP_V13.6, JP2.5, JP2.6, Q1.2, R11.1, S1.1, S1.2, U2.21, U2.3, U2.5, U3.2
- net RAW: now also C19.1, U3.1, U3.3
