File: eagle/Segment16Keyboard.brd (EAGLE design)
At the start: 52.1 x 26.7 mm, 21 parts, among them Q1 16MHZ, U1 LCD-16X2NOHOLES, U2 ATMEGA328, U3 MIC5205

Commit message: Board V1
Parts:
- LED1: value Red -> RED
Connections:
- net D12 renamed E
- net D13 renamed RS
- net D4 renamed DB7
- net D5 renamed DB6
- net D6 renamed DB5
- net D7 renamed DB4
- net N$14 renamed A
- net N$5 renamed VO
Routing:
- net GND: track 16.5 -> 15.7 mm, vias 9 -> 10
Other:
- outline, holes or cut-outs redrawn
- board text added: "A"
- board text added: "DB4"
- board text added: "DB5"
- board text added: "DB6"
- board text added: "DB7"
- board text added: "DTR"
- board text added: "E"
- board text added: "GND"
- board text added: "MISO"
- board text added: "MOSI"
- board text added: "N/C"
- board text added: "RAW"
- board text added: "RESET"
- board text added: "RS"
- board text added: "RXI"
- board text added: "SCK"
- board text added: "TXO"
- board text added: "V0"
- board text added: "V1"
- board text added: "VCC"
- board text removed: "REV -"
