File: eagle/Segment16Keyboard.sch (EAGLE design)
At the start: 6 parts, among them U1 LCD-16X2NOHOLES

Commit message: WIP
Parts:
- added C1, C2, C3: 0.1uF, adafruit:C-USC0805
- added C10: 0.1uF, resistor:C-USC0805
- added C13, C19: 10uF, resistor:C-USC0805
- added D3: Green, adafruit:LEDCHIPLED_0805
- added ISP_V13: (no value), SparkFun-Connectors:M06SIP
- added JP2: FTDI Basic, SparkFun:ARDUINO_SERIAL_PROGRAMPTH
- added LED1: Red, Testing:LED
- added Q1: 16MHZ, SparkFun-FreqCtrl:RESONATOR16MHZ
- added R11: 10K, SparkFun:RESISTOR0603-RES
- added R2: 10K, adafruit:R-US_M0805
- added R6: 300, adafruit:R-US_M0805
- added S1: Reset, Testing:SWITCH-MOMENTARY-2SMD-ALT01
- added SJ1: SOLDERJUMPERNC, SparkFun-Passives:SOLDERJUMPERNC
- added U2: ATMEGA328, SparkFun:ATMEGA168
- added U3: MIC5205, SparkFun:V_REG_LDOSMD
Connections:
- new net A0: U2.PC0(ADC0)
- new net A1: U2.PC1(ADC1)
- new net A2: U2.PC2(ADC2)
- new net A3: U2.PC3(ADC3)
- new net A4: U2.PC4(ADC4/SDA)
- new net A5: U2.PC5(ADC5/SCL)
- new net A6: U2.ADC6
- new net A7: U2.ADC7
- new net AREF: C1.2, U2.AREF
- new net D10: U2.PB2(SS/OC1B)
- new net D2: U2.PD2(INT0)
- new net D3: U2.PD3(INT1)
- new net D4: U2.PD4(XCK/T0)
- new net D5: U2.PD5(T1)
- new net D6: U2.PD6(AIN0)
- new net D7: U2.PD7(AIN1)
- new net DTR: C2.2, JP2.DTR
- new net MISO: ISP_V13.3, U2.PB4(MISO)
- new net MOSI: ISP_V13.2, U2.PB3(MOSI/OC2)
- new net N$12: D3.A, R6.2
- new net N$13: Q1.3, U2.PB7(XTAL2/TOSC2)
- new net N$15: Q1.1, U2.PB6(XTAL1/TOSC1)
- new net N$19: LED1.A, SJ1.1, U3.OUT
- new net N$20: LED1.C, R11.2
- new net RESET: C2.1, ISP_V13.1, R2.1, S1.2, U2.PC6(/RESET)
- new net RXI: JP2.TXO, U2.PD0(RXD)
- new net SCK: ISP_V13.5, R6.1, U2.PB5(SCK)
- new net SSRX: U2.PB0(ICP)
- new net SSTX: U2.PB1(OC1A)
- new net TXO: JP2.RXI, U2.PD1(TXD)
- new net VCC: C10.1, C13.1, C3.2, ISP_V13.4, JP2.VCC, R2.2, SJ1.2, U2.AVCC, U2.VCC@1, U2.VCC@2
- net GND: now also C1.1, C10.2, C13.2, C19.2, C3.1, D3.C, ISP_V13.6, JP2.CTS, JP2.GND, Q1.2, R11.1, S1.1, U2.AGND, U2.GND@1, U2.GND@2, U3.GND
- net RAW: now also C19.1, U3.EN, U3.IN
Other:
- note added: "(for low power aplications)"
- note added: "Board is marked with combination of"
- note added: "Max Current Output: 150mA"
- note added: "Max Voltage Input: 16VDC"
- note added: "Power isolation jumper"
- note added: "VCC = 5V or 3.3V Output"
- note added: "resonator frequency and regulator voltage."
