File: eagle/Segment16Keyboard.sch (EAGLE design)
At the start: 21 parts, among them Q1 16MHZ, U1 LCD-16X2NOHOLES, U2 ATMEGA328, U3 MIC5205

Commit message: Board V1
Parts:
- LED1: value Red -> RED
Connections:
- net D12 renamed E
- net D13 renamed RS
- net D4 renamed DB7
- net D5 renamed DB6
- net D6 renamed DB5
- net D7 renamed DB4
- net N$14 renamed A
- net N$5 renamed VO
Other:
- moved on the sheet: BRGT
Changed lines of the file:
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@@
 <clearance class="0" value="0.254"/>
 </class>
-<class number="1" name="vcc" width="0.508" drill="0.381">
+<class number="1" name="vcc" width="0.508" drill="0.508">
 <clearance class="1" value="0.254"/>
 </class>
-<class number="2" name="raw" width="0.508" drill="0.381">
+<class number="2" name="raw" width="0.508" drill="0.508">
 <clearance class="2" value="0.254"/>
 </class>
@@
 <part name="GND25" library="SparkFun" deviceset="GND" device=""/>
 <part name="R11" library="adafruit" deviceset="R-US_" device="R0805" value="10K"/>
-<part name="LED1" library="Testing" deviceset="LED" device="" value="Red"/>
+<part name="LED1" library="Testing" deviceset="LED" device="" value="RED"/>
 <part name="GND28" library="SparkFun" deviceset="GND" device=""/>
 <part name="U3" library="SparkFun" deviceset="V_REG_LDO" device="SMD" value="MIC5205"/>
@@
 <instance part="CTRST" gate="G$1" x="111.76" y="119.38" rot="R270"/>
 <instance part="GND4" gate="1" x="124.46" y="63.5"/>
-<instance part="BRGT" gate="G$1" x="116.84" y="68.58"/>
+<instance part="BRGT" gate="G$1" x="109.22" y="68.58"/>
 <instance part="R2" gate="G$1" x="177.8" y="129.54" rot="R90"/>
 <instance part="GND5" gate="1" x="177.8" y="104.14"/>
@@
 </segment>
 </net>
-<net name="N$5" class="0">
+<net name="VO" class="0">
 <segment>
 <pinref part="CTRST" gate="G$1" pin="S"/>
@@
 </segment>
 </net>
-<net name="D13" class="0">
+<net name="RS" class="0">
 <segment>
 <pinref part="U1" gate="G$1" pin="RS"/>
@@
 </segment>
 </net>
-<net name="D12" class="0">
+<net name="E" class="0">
 <segment>
 <pinref part="U1" gate="G$1" pin="E"/>
@@
 </segment>
 </net>
-<net name="N$14" class="0">
+<net name="A" class="0">
 <segment>
 <pinref part="BRGT" gate="G$1" pin="S"/>
-<wire x1="121.92" y1="68.58" x2="121.92" y2="76.2" width="0.1524" layer="91"/>
+<wire x1="114.3" y1="68.58" x2="114.3" y2="76.2" width="0.1524" layer="91"/>
 <pinref part="U1" gate="G$1" pin="A"/>
-<wire x1="121.92" y1="76.2" x2="124.46" y2="76.2" width="0.1524" layer="91"/>
+<wire x1="114.3" y1="76.2" x2="124.46" y2="76.2" width="0.1524" layer="91"/>
 </segment>
 </net>
@@
 <segment>
 <pinref part="BRGT" gate="G$1" pin="E"/>
-<wire x1="116.84" y1="73.66" x2="116.84" y2="76.2" width="0.1524" layer="91"/>
-<wire x1="116.84" y1="76.2" x2="114.3" y2="76.2" width="0.1524" layer="91"/>
-<label x="114.3" y="76.2" size="1.27" layer="95" rot="R180" xref="yes"/>
+<wire x1="109.22" y1="73.66" x2="109.22" y2="76.2" width="0.1524" layer="91"/>
+<wire x1="109.22" y1="76.2" x2="106.68" y2="76.2" width="0.1524" layer="91"/>
+<label x="106.68" y="76.2" size="1.27" layer="95" rot="R180" xref="yes"/>
 </segment>
 </net>
@@
 </segment>
 </net>
-<net name="D7" class="0">
+<net name="DB4" class="0">
 <segment>
 <wire x1="251.46" y1="81.28" x2="254" y2="81.28" width="0.1524" layer="91"/>
@@
 </segment>
 </net>
-<net name="D4" class="0">
+<net name="DB7" class="0">
 <segment>
 <wire x1="251.46" y1="88.9" x2="254" y2="88.9" width="0.1524" layer="91"/>
@@
 </segment>
 </net>
-<net name="D5" class="0">
+<net name="DB5" class="0">
+<segment>
+<wire x1="251.46" y1="83.82" x2="254" y2="83.82" width="0.1524" layer="91"/>
+<pinref part="U2" gate="G$1" pin="PD6(AIN0)"/>
+<label x="254" y="83.82" size="1.27" layer="95" xref="yes"/>
+</segment>
+<segment>
+<pinref part="U1" gate="G$1" pin="DB5"/>
+<wire x1="124.46" y1="83.82" x2="121.92" y2="83.82" width="0.1524" layer="91"/>
+<label x="121.92" y="83.82" size="1.27" layer="95" rot="R180" xref="yes"/>
+</segment>
+</net>
+<net name="A3" class="0">
+<segment>
+<pinref part="U2" gate="G$1" pin="PC3(ADC3)"/>
+<wire x1="251.46" y1="114.3" x2="254" y2="114.3" width="0.1524" layer="91"/>
+<label x="254" y="114.3" size="1.27" layer="95" xref="yes"/>
+</segment>
+</net>
+<net name="D2" class="0">
+<segment>
+<pinref part="U2" gate="G$1" pin="PD2(INT0)"/>
+<wire x1="251.46" y1="93.98" x2="254" y2="93.98" width="0.1524" layer="91"/>
+<label x="254" y="93.98" size="1.27" layer="95" xref="yes"/>
+</segment>
+<segment>
+<pinref part="U$2" gate="G$1" pin="5"/>
+<wire x1="48.26" y1="93.98" x2="55.88" y2="93.98" width="0.1524" layer="91"/>
+<label x="55.88" y="93.98" size="1.27" layer="95" xref="yes"/>
+</segment>
+</net>
+<net name="D3" class="0">
+<segment>
+<pinref part="U2" gate="G$1" pin="PD3(INT1)"/>
+<wire x1="251.46" y1="91.44" x2="254" y2="91.44" width="0.1524" layer="91"/>
+<label x="254" y="91.44" size="1.27" layer="95" xref="yes"/>
+</segment>
+<segment>
+<pinref part="U$2" gate="G$1" pin="1"/>
+<wire x1="48.26" y1="83.82" x2="58.42" y2="83.82" width="0.1524" layer="91"/>
+<label x="58.42" y="83.82" size="1.27" layer="95" xref="yes"/>
+</segment>
+</net>
+<net name="N$20" class="0">
+<segment>
+<pinref part="R11" gate="G$1" pin="2"/>
+<pinref part="LED1" gate="G$1" pin="C"/>
+<wire x1="104.14" y1="170.18" x2="104.14" y2="167.64" width="0.1524" layer="91"/>
+</segment>
+</net>
+<net name="DB6" class="0">
+<segment>
+<pinref part="U1" gate="G$1" pin="DB6"/>
+<wire x1="121.92" y1="81.28" x2="124.46" y2="81.28" width="0.1524" layer="91"/>
+<label x="121.92" y="81.28" size="1.27" layer="95" rot="R180" xref="yes"/>
+</segment>
 <segment>
 <wire x1="251.46" y1="86.36" x2="254" y2="86.36" width="0.1524" layer="91"/>
@@
 <label x="254" y="86.36" size="1.27" layer="95" xref="yes"/>
 </segment>
-<segment>
-<pinref part="U1" gate="G$1" pin="DB6"/>
-<wire x1="121.92" y1="81.28" x2="124.46" y2="81.28" width="0.1524" layer="91"/>
-<label x="121.92" y="81.28" size="1.27" layer="95" rot="R180" xref="yes"/>
-</segment>
-</net>
-<net name="D6" class="0">
-<segment>
-<wire x1="251.46" y1="83.82" x2="254" y2="83.82" width="0.1524" layer="91"/>
-<pinref part="U2" gate="G$1" pin="PD6(AIN0)"/>
-<label x="254" y="83.82" size="1.27" layer="95" xref="yes"/>
-</segment>
-<segment>
-<pinref part="U1" gate="G$1" pin="DB5"/>
-<wire x1="124.46" y1="83.82" x2="121.92" y2="83.82" width="0.1524" layer="91"/>
-<label x="121.92" y="83.82" size="1.27" layer="95" rot="R180" xref="yes"/>
-</segment>
-</net>
-<net name="A3" class="0">
-<segment>
-<pinref part="U2" gate="G$1" pin="PC3(ADC3)"/>
-<wire x1="251.46" y1="114.3" x2="254" y2="114.3" width="0.1524" layer="91"/>
-<label x="254" y="114.3" size="1.27" layer="95" xref="yes"/>
-</segment>
-</net>
-<net name="D2" class="0">
-<segment>
-<pinref part="U2" gate="G$1" pin="PD2(INT0)"/>
-<wire x1="251.46" y1="93.98" x2="254" y2="93.98" width="0.1524" layer="91"/>
-<label x="254" y="93.98" size="1.27" layer="95" xref="yes"/>
-</segment>
-<segment>
-<pinref part="U$2" gate="G$1" pin="5"/>
-<wire x1="48.26" y1="93.98" x2="55.88" y2="93.98" width="0.1524" layer="91"/>
-<label x="55.88" y="93.98" size="1.27" layer="95" xref="yes"/>
-</segment>
-</net>
-<net name="D3" class="0">
-<segment>
-<pinref part="U2" gate="G$1" pin="PD3(INT1)"/>
-<wire x1="251.46" y1="91.44" x2="254" y2="91.44" width="0.1524" layer="91"/>
-<label x="254" y="91.44" size="1.27" layer="95" xref="yes"/>
-</segment>
-<segment>
-<pinref part="U$2" gate="G$1" pin="1"/>
-<wire x1="48.26" y1="83.82" x2="58.42" y2="83.82" width="0.1524" layer="91"/>
-<label x="58.42" y="83.82" size="1.27" layer="95" xref="yes"/>
-</segment>
-</net>
-<net name="N$20" class="0">
-<segment>
-<pinref part="R11" gate="G$1" pin="2"/>
-<pinref part="LED1" gate="G$1" pin="C"/>
-<wire x1="104.14" y1="170.18" x2="104.14" y2="167.64" width="0.1524" layer="91"/>
-</segment>
-</net>
+</net>
